File: pcb/obd2_logger/obd2_logger.kicad_pcb (KiCad board)
At the start: 2 copper layers, 80 x 56 mm, 14 parts

Commit message: Improve pcb
Parts:
- removed ? (x4): , MountingHole_3.2mm_M3
- added MH1: MountingHole, MountingHole_3.2mm_M3, F.Cu at (54.5, 42.5)
- added MH2: MountingHole, MountingHole_3.2mm_M3, F.Cu at (127.5, 42.5)
- added MH3: MountingHole, MountingHole_3.2mm_M3, F.Cu at (54.5, 91.5)
- added MH4: MountingHole, MountingHole_3.2mm_M3, F.Cu at (127.5, 91.5)
- moved J_RTC 66.9 mm to (112.5, 48.5)
- moved J_ESP32_L 64.2 mm to (59.0, 44.0)
- moved J_ESP32_R 64.2 mm to (81.9, 44.0)
- moved J_OBD2 64.2 mm to (97.0, 87.0)
- moved J_OLED 64.2 mm to (97.0, 53.0)
- moved R1 64.2 mm to (101.0, 67.0)
- moved R2 64.2 mm to (101.0, 72.0)
- moved J_CAN_5V 59.7 mm to (120.0, 56.9)
- moved J_CAN_3V3 59.4 mm to (120.0, 72.4)
- moved J_SD 59.3 mm to (89.8, 43.5)
Routing:
- net VCC_5V: track 176.9 -> 15.5 mm
- net GND: track 292.1 -> 132.7 mm, vias 9 -> 0
- net I2C_SCL: track 54.2 -> 11.1 mm, vias 0 -> 1
- net I2C_SDA: track 51.4 -> 11.8 mm, vias 0 -> 1
- net SD_MISO: track 34.4 -> 48.6 mm
- net SD_SCK: track 42.0 -> 33.7 mm
- net CAN_RX_5V: track 30.9 -> 28.3 mm
- net VCC_3V3: track 157.9 -> 156.0 mm, vias 0 -> 1
- net CAN_RX: track 62.3 -> 61.5 mm, vias 0 -> 2
- net SD_CS: track 59.8 -> 60.0 mm, vias 2 -> 1
